Commit message: feat: add one-goal real robot flow

File: MiniChallenge6/puzzlebot_sim/urdf/puzzlebot.urdf (robot description, URDF)
Before this commit: robot puzzlebot, 5 links, 4 joints
Links:
- removed link caster_link
- removed link wheel_l_link
- removed link wheel_r_link
- added link camera; visual box size=0.03 0.04 0.03
- added link camera_optical_frame
- added link caster, mass 0.1; collision mesh filename=package://minic3/meshes/Puzzlebot_Caster_Wheel.stl scale=1 1 1; visual mesh filename=package://minic3/meshes/Puzzlebot_Caster_Wheel.stl scale=1 1 1
- added link laser; visual cylinder length=0.03 radius=0.035
- added link wheel_l, mass 0.3; collision mesh filename=package://minic3/meshes/Puzzlebot_Wheel.stl scale=1 1 1; visual mesh filename=package://minic3/meshes/Puzzlebot_Wheel.stl scale=1 1 1
- added link wheel_r, mass 0.3; collision mesh filename=package://minic3/meshes/Puzzlebot_Wheel.stl scale=1 1 1; visual mesh filename=package://minic3/meshes/Puzzlebot_Wheel.stl scale=1 1 1
- link base_link: mass None -> 1.0; geometry collision mesh filename=package://minic3/meshes/Puzzlebot_Jetson_Lidar_Edition_Base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 scale=1 1 1; visual mesh filename=package://minic3/meshes/Puzzlebot_Jetson_Lidar_Edition_Base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 scale=1 1 1
Joints:
- added joint camera_joint: type fixed, parent base_link, child camera, origin xyz=0.10 0.0 0.12 rpy=0.0 0.0 0.0
- added joint camera_optical_joint: type fixed, parent camera, child camera_optical_frame, origin xyz=0 0 0 rpy=-1.5708 0 -1.5708
- added joint laser_joint: type fixed, parent base_link, child laser, origin xyz=0.08 0.0 0.09 rpy=0.0 0.0 0.0
- joint caster_joint: child caster_link -> caster; origin xyz=-0.095 0.0 -0.03 rpy=0.0 0.0 0.0 -> xyz=-0.09 0 -0.043 rpy=0.0 0.0 0.0
- joint wheel_l_joint: axis 0 1 0 -> 0.0 1.0 0.0; child wheel_l_link -> wheel_l
- joint wheel_r_joint: axis 0 1 0 -> 0.0 1.0 0.0; child wheel_r_link -> wheel_r
